File: Hardware/Counter/Counter.kicad_pcb (KiCad board)
At the start: 2 copper layers, 100 x 100 mm, 241 parts, among them J1 PWR, J2 OUT, Q1 FDN360P, Q10 FDN335N, Q100 FDN335N, Q101 FDN360P, Q102 FDN335N, Q103 FDN335N, Q104 FDN335N, Q105 FDN360P, Q106 FDN335N, Q107 FDN335N, Q108 FDN335N, Q109 FDN335N, Q11 FDN335N, Q110 FDN360P, Q111 FDN335N, Q112 FDN335N, Q113 FDN360P, Q114 FDN335N, Q115 FDN335N, Q116 FDN335N, Q117 FDN335N, Q118 FDN360P, Q119 FDN335N, Q12 FDN335N, Q120 FDN335N, Q121 FDN360P, Q122 FDN335N, Q123 FDN335N, Q124 FDN335N, Q125 FDN335N, Q126 FDN360P, Q127 FDN335N, Q128 FDN335N, Q129 FDN335N, Q13 FDN360P, Q130 FDN335N, Q131 FDN335N, Q132 FDN335N, Q133 FDN335N, Q134 FDN335N, Q135 FDN335N, Q136 FDN335N, Q14 FDN360P, Q15 FDN360P, Q16 FDN335N, Q17 FDN335N, Q18 FDN335N, Q19 FDN335N, Q2 FDN360P, Q20 FDN335N, Q21 FDN360P, Q22 FDN360P, Q23 FDN360P, Q24 FDN335N, Q25 FDN335N, Q26 FDN335N, Q27 FDN335N, Q28 FDN335N, Q29 FDN335N, Q3 FDN335N, Q30 FDN360P, Q31 FDN335N, Q32 FDN335N, Q33 FDN335N, Q34 FDN360P, Q35 FDN335N, Q36 FDN335N, Q37 FDN360P, Q38 FDN335N, Q39 FDN335N, Q4 FDN335N, Q40 FDN335N, Q41 FDN335N, Q42 FDN360P, Q43 FDN335N, Q44 FDN335N, Q45 FDN360P, Q46 FDN335N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

Commit message: working on bit 2
Parts:
- moved Q102 201.4 mm to (45.5, 44.0), turned to 90 degrees
- moved Q101 197.2 mm to (45.5, 40.5), turned to 90 degrees
- moved Q104 193.5 mm to (49.0, 47.5), turned to 90 degrees
- moved Q103 192.6 mm to (45.5, 47.5), turned to 90 degrees
- moved U58 190.4 mm to (49.0, 40.5), turned to 90 degrees
- moved U59 189.0 mm to (49.0, 44.0), turned to 90 degrees
- moved Q106 161.9 mm to (45.5, 56.0), turned to 90 degrees
- moved Q105 158.4 mm to (45.5, 52.5), turned to 90 degrees
- moved Q117 156.3 mm to (53.0, 56.0), turned to 90 degrees
- moved Q108 154.4 mm to (49.0, 59.5), turned to 90 degrees
- moved Q124 153.6 mm to (56.5, 56.0), turned to 90 degrees
- moved Q107 153.5 mm to (45.5, 59.5), turned to 90 degrees
- moved U60 153.4 mm to (49.0, 52.5), turned to 90 degrees
- moved U61 149.8 mm to (49.0, 56.0), turned to 90 degrees
- moved U69 149.4 mm to (56.5, 52.5), turned to 90 degrees
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Routing:
- net /XOR1/!A: track 0.00 -> 23.5 mm
- net /B1: track 0.00 -> 20.1 mm, vias 0 -> 2
- net /Q_17: track 0.00 -> 17.7 mm, vias 0 -> 4
- net /XOR1/!B: track 0.00 -> 16.9 mm, vias 0 -> 2
- net /Q_18: track 0.00 -> 15.0 mm
- net Net-(Q105-Pad2): track 0.00 -> 12.8 mm
- net Net-(Q101-Pad2): track 0.00 -> 12.8 mm
- net /DW: track 2.52 -> 14.3 mm
- net /B0: track 13.3 -> 24.0 mm
- net /!B0: track 50.7 -> 60.7 mm, vias 2 -> 3
- net GND: track 14.0 -> 19.8 mm, vias 10 -> 16
- net Net-(Q114-Pad2): track 0.00 -> 5.22 mm
- net Net-(Q29-Pad3): track 12.3 -> 8.89 mm
- net Net-(Q113-Pad3): track 0.00 -> 3.38 mm
- net Net-(Q111-Pad2): track 0.00 -> 3.38 mm
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
Commit message: bit 2 complete
Parts:
- moved Q126 170.2 mm to (79.0, 44.5), turned to 90 degrees
- moved Q125 169.3 mm to (75.5, 48.0), turned to 90 degrees
- moved U71 169.3 mm to (75.5, 51.5), turned to 90 degrees
- moved U70 164.7 mm to (75.5, 44.5), turned to 90 degrees
- moved Q127 161.4 mm to (79.0, 48.0), turned to 90 degrees
- moved Q128 161.2 mm to (79.0, 51.5), turned to 90 degrees
- moved U76 86.7 mm to (86.5, 46.0), turned to 90 degrees
- moved Q132 86.4 mm to (83.0, 49.5), turned to 90 degrees
- moved U75 84.3 mm to (83.0, 46.0), turned to 90 degrees
- moved Q134 84.1 mm to (90.0, 49.5), turned to 90 degrees
- moved Q133 83.3 mm to (86.5, 49.5), turned to 90 degrees
- moved Q135 78.1 mm to (97.0, 49.5), turned to 90 degrees
- moved U77 76.0 mm to (90.0, 46.0), turned to 90 degrees
- moved U79 74.5 mm to (93.5, 46.0), turned to 90 degrees
- moved U78 73.8 mm to (97.0, 46.0), turned to 90 degrees
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Routing:
- net /B1: track 20.1 -> 55.8 mm, vias 2 -> 7
- net /Q_19: track 0.00 -> 26.3 mm, vias 0 -> 2
- net /CLK: track 74.0 -> 99.2 mm
- net /Q_16: track 1.89 -> 26.4 mm, vias 0 -> 2
- net /XOR2/!A: track 0.00 -> 23.5 mm
- net /!B1: track 0.00 -> 22.3 mm, vias 0 -> 3
- net Net-(Q133-Pad3): track 0.00 -> 21.3 mm
- net /FF2/!CLK: track 0.00 -> 17.9 mm
- net /XOR2/!B: track 0.00 -> 16.9 mm, vias 0 -> 2
- net Net-(Q125-Pad3): track 0.00 -> 15.9 mm
- net /Q_18: track 15.0 -> 28.7 mm
- net /Q_20: track 0.00 -> 13.3 mm
- net GND: track 19.8 -> 29.5 mm, vias 16 -> 26
- net Net-(Q122-Pad2): track 0.00 -> 5.22 mm
- net Net-(Q126-Pad3): track 0.00 -> 3.38 mm
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
Commit message: bit 3 complete
Parts:
- removed R11, R12, R13: 10K, Resistor_SMD:R_0805_2012Metric
- added SW3: SW_Push, Button_Switch_SMD:SW_SPST_TL3342, F.Cu at (173.0, 32.5)
- moved Q14 194.4 mm to (49.0, 91.5), turned to 90 degrees
- moved Q13 191.9 mm to (45.5, 91.5), turned to 90 degrees
- moved Q16 187.4 mm to (45.5, 95.0), turned to 90 degrees
- moved Q73 186.6 mm to (82.5, 70.5), turned to 90 degrees
- moved Q72 186.2 mm to (79.0, 74.0), turned to 90 degrees
- moved U34 186.0 mm to (79.0, 77.5), turned to 90 degrees
- moved Q17 185.6 mm to (49.0, 95.0), turned to 90 degrees
- moved Q20 181.7 mm to (59.5, 95.0), turned to 90 degrees
- moved Q19 180.8 mm to (56.0, 95.0), turned to 90 degrees
- moved U33 180.6 mm to (79.0, 70.5), turned to 90 degrees
- moved Q18 180.0 mm to (52.5, 95.0), turned to 90 degrees
- moved Q74 178.4 mm to (82.5, 74.0), turned to 90 degrees
- moved Q75 177.5 mm to (82.5, 77.5), turned to 90 degrees
- moved U7 177.2 mm to (59.5, 91.5), turned to 90 degrees
- moved Q15 175.4 mm to (52.5, 91.5), turned to 90 degrees
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Connections:
- Q104 pad 3: /Q_17 -> /Q
- Q108 pad 3: /Q_16 -> /Q_20
- Q109 pad 1: /Q_17 -> /Q
- Q110 pad 1: /Q_17 -> /Q
- Q110 pad 2: /Q_18 -> /Q_16
- Q111 pad 3: /Q_18 -> /Q_16
- Q113 pad 2: /Q_18 -> /Q_16
- Q114 pad 3: /Q_18 -> /Q_16
- Q118 pad 2: /Q_19 -> /Q_17
- Q119 pad 1: /Q_16 -> /Q_20
- Q119 pad 3: /Q_19 -> /Q_17
- Q12 pad 3: /Q_2 -> /Q_4
- Q120 pad 1: /Q_16 -> /Q_20
- Q121 pad 2: /Q_19 -> /Q_17
- Q122 pad 3: /Q_19 -> /Q_17
- Q124 pad 1: /Q_16 -> /Q_20
- Q125 pad 1: /Q_19 -> /Q_17
- Q126 pad 1: /Q_19 -> /Q_17
- Q127 pad 1: /Q_18 -> /Q_16
- Q128 pad 3: /Q -> /Q_19
- Q130 pad 2: /Q -> /Q_19
- Q130 pad 3: /Q_20 -> /Q_18
- Q131 pad 3: /Q_20 -> /Q_18
- Q133 pad 2: /Q_20 -> /Q_18
- Q20 pad 3: /Q_7 -> /Q_9
- Q28 pad 3: /Q_6 -> /Q_8
- Q32 pad 3: /Q_3 -> /Q_5
- Q33 pad 1: /Q_1 -> /Q_3
- Q34 pad 1: /Q_1 -> /Q_3
- Q34 pad 2: /Q_4 -> /Q_6
- Q35 pad 3: /Q_4 -> /Q_6
- Q37 pad 2: /Q_4 -> /Q_6
- Q38 pad 3: /Q_4 -> /Q_6
- Q42 pad 2: /Q_5 -> /Q_7
- Q43 pad 1: /Q_2 -> /Q_4
- Q43 pad 3: /Q_5 -> /Q_7
- Q44 pad 1: /Q_2 -> /Q_4
- Q45 pad 2: /Q_5 -> /Q_7
- Q46 pad 3: /Q_5 -> /Q_7
- Q48 pad 1: /Q_2 -> /Q_4
- Q49 pad 1: /Q_7 -> /Q_9
- Q50 pad 1: /Q_7 -> /Q_9
- Q50 pad 2: /Q_8 -> /Q_10
- Q51 pad 3: /Q_8 -> /Q_10
- Q53 pad 2: /Q_8 -> /Q_10
- Q54 pad 3: /Q_8 -> /Q_10
- Q58 pad 2: /Q_9 -> /Q_11
- Q59 pad 1: /Q_6 -> /Q_8
- Q59 pad 3: /Q_9 -> /Q_11
- Q6 pad 3: /Q_1 -> /Q_3
- Q60 pad 1: /Q_6 -> /Q_8
- Q61 pad 2: /Q_9 -> /Q_11
- Q62 pad 3: /Q_9 -> /Q_11
- Q64 pad 1: /Q_6 -> /Q_8
- Q65 pad 1: /Q_3 -> /Q_5
- Q66 pad 1: /Q_3 -> /Q_5
- Q68 pad 3: /Q_10 -> /Q_12
- Q70 pad 2: /Q_10 -> /Q_12
- Q70 pad 3: /Q_12 -> /Q_14
- Q71 pad 3: /Q_12 -> /Q_14
- Q72 pad 1: /Q_5 -> /Q_7
- Q73 pad 1: /Q_5 -> /Q_7
- Q74 pad 1: /Q_4 -> /Q_6
- Q75 pad 3: /Q_11 -> /Q_13
- Q76 pad 1: /Q_9 -> /Q_11
- Q77 pad 1: /Q_9 -> /Q_11
- Q78 pad 1: /Q_8 -> /Q_10
- Q79 pad 3: /Q_14 -> /Q_15
- Q81 pad 2: /Q_11 -> /Q_13
- Q81 pad 3: /Q_15 -> /Q_2
- Q82 pad 3: /Q_15 -> /Q_2
- Q84 pad 2: /Q_14 -> /Q_15
- Q84 pad 3: /Q_13 -> /Q_1
- Q85 pad 3: /Q_13 -> /Q_1
- Q87 pad 2: /Q_12 -> /Q_14
- Q92 pad 2: /Q_15 -> /Q_2
- Q97 pad 2: /Q_13 -> /Q_1
- U11 pad 2: /Q_3 -> /Q_5
- U12 pad 1: /Q_1 -> /Q_3
- U18 pad 1: /Q_2 -> /Q_4
- U19 pad 1: /Q_2 -> /Q_4
- U20 pad 1: /Q_7 -> /Q_9
- U26 pad 1: /Q_6 -> /Q_8
- U27 pad 1: /Q_6 -> /Q_8
- U29 pad 2: /Q_10 -> /Q_12
- U3 pad 2: /Q_1 -> /Q_3
- U31 pad 2: /Q_12 -> /Q_14
- U31 pad 3: /Q_10 -> /Q_12
- U32 pad 2: /Q_12 -> /Q_14
- U33 pad 1: /Q_4 -> /Q_6
- U34 pad 2: /Q_11 -> /Q_13
- U35 pad 1: /Q_8 -> /Q_10
- U36 pad 2: /Q_14 -> /Q_15
- U38 pad 2: /Q_15 -> /Q_2
- U38 pad 3: /Q_11 -> /Q_13
- U39 pad 2: /Q_15 -> /Q_2
- U41 pad 2: /Q_13 -> /Q_1
- U41 pad 3: /Q_14 -> /Q_15
- U42 pad 2: /Q_13 -> /Q_1
- U44 pad 3: /Q_12 -> /Q_14
- U49 pad 3: /Q_15 -> /Q_2
- U5 pad 2: /Q_2 -> /Q_4
- U54 pad 3: /Q_13 -> /Q_1
- U59 pad 2: /Q_17 -> /Q
- U61 pad 2: /Q_16 -> /Q_20
- U62 pad 1: /Q_17 -> /Q
- U68 pad 1: /Q_16 -> /Q_20
- U69 pad 1: /Q_16 -> /Q_20
- U7 pad 2: /Q_7 -> /Q_9
- U70 pad 1: /Q_18 -> /Q_16
- U71 pad 2: /Q -> /Q_19
- U73 pad 2: /Q_20 -> /Q_18
- U73 pad 3: /Q -> /Q_19
- U74 pad 2: /Q_20 -> /Q_18
- U76 pad 3: /Q_20 -> /Q_18
- U9 pad 2: /Q_6 -> /Q_8
Routing:
- net /B2: track 0.00 -> 48.9 mm, vias 0 -> 2
- net /RST: track 25.7 -> 68.2 mm
- net /Q_6: track 0.00 -> 30.7 mm
- net /Q_14: track 0.00 -> 30.3 mm
- net /Q_2: track 0.00 -> 28.5 mm
- net /Q_7: track 0.00 -> 28.1 mm, vias 0 -> 2
- net /XOR4/!A: track 0.00 -> 26.7 mm, vias 0 -> 2
- net /!B2: track 0.00 -> 25.8 mm, vias 0 -> 5
- net /XOR3/!A: track 0.00 -> 25.8 mm, vias 0 -> 2
- net /XOR4/!B: track 0.00 -> 25.7 mm, vias 0 -> 2
- net /CLK: track 99.2 -> 124.3 mm
- net GND: track 29.5 -> 54.6 mm, vias 26 -> 52
- net /Q_4: track 0.00 -> 23.8 mm
- net Net-(Q92-Pad3): track 0.00 -> 21.3 mm
- net /XOR3/!B: track 0.00 -> 19.2 mm, vias 0 -> 2
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
Commit message: working on connectin bits together
Parts:
- moved U41 185.4 mm to (76.6, 92.9), turned to 90 degrees
- moved Q84 178.5 mm to (76.6, 96.4), turned to 90 degrees
- moved Q83 177.6 mm to (80.1, 96.4), turned to 90 degrees
- moved U42 176.2 mm to (83.6, 96.4), turned to 90 degrees
- moved U40 170.6 mm to (80.1, 92.9), turned to 90 degrees
- moved Q85 168.9 mm to (83.6, 92.9), turned to 90 degrees
- moved Q77 159.6 mm to (72.6, 91.9), turned to 90 degrees
- moved Q76 159.4 mm to (69.1, 95.4), turned to 90 degrees
- moved U36 159.2 mm to (69.1, 98.9), turned to 90 degrees
- moved U35 153.4 mm to (69.1, 91.9), turned to 90 degrees
- moved Q78 151.7 mm to (72.6, 95.4), turned to 90 degrees
- moved Q79 150.5 mm to (72.6, 98.9), turned to 90 degrees
- moved Q64 130.7 mm to (46.3, 102.5), turned to 90 degrees
- moved Q57 127.9 mm to (46.3, 99.0), turned to 90 degrees
- moved U27 125.3 mm to (49.8, 102.5), turned to 90 degrees
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Connections:
- Q2 pad 1: /UP -> /B1
- Q8 pad 1: /DW -> /!B1
- U2 pad 1: /B1 -> /UP
- U4 pad 1: /!B1 -> /DW
Routing:
- net /B3: track 0.00 -> 45.3 mm
- net /Q_10: track 0.00 -> 33.6 mm
- net /Q_1: track 0.00 -> 28.5 mm
- net /Q_11: track 0.00 -> 28.1 mm, vias 0 -> 2
- net /XOR6/!A: track 0.00 -> 26.7 mm, vias 0 -> 2
- net /XOR5/!A: track 0.00 -> 26.7 mm, vias 0 -> 2
- net /XOR6/!B: track 0.00 -> 25.7 mm, vias 0 -> 2
- net /XOR5/!B: track 0.00 -> 25.7 mm, vias 0 -> 2
- net /!B3: track 0.00 -> 22.3 mm, vias 0 -> 3
- net /Q_8: track 1.89 -> 23.8 mm
- net /RST: track 68.2 -> 90.0 mm
- net Net-(Q97-Pad3): track 0.00 -> 21.3 mm
- net GND: track 54.6 -> 74.3 mm, vias 52 -> 71
- net /FF4/!CLK: track 0.00 -> 17.9 mm
- net /Q_9: track 1.89 -> 18.0 mm
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
Commit message: layout complete- gerbers generated
Parts:
- moved SW3 156.4 mm to (17.0, 43.0), turned to 90 degrees
- moved R10 153.0 mm to (21.0, 43.0), turned to 90 degrees
- moved R9 120.6 mm to (36.8, 17.8), turned to -90 degrees
- moved D6 117.9 mm to (36.8, 14.0), turned to 90 degrees
- moved R7 97.8 mm to (99.1, 101.6), turned to 90 degrees
- moved D2 95.5 mm to (104.1, 105.4), turned to -90 degrees
- moved R5 93.9 mm to (101.6, 101.6), turned to 90 degrees
- moved J2 87.3 mm to (109.2, 109.5), turned to -90 degrees
- moved D1 85.1 mm to (106.7, 105.4), turned to -90 degrees
- moved D4 79.2 mm to (99.1, 105.4), turned to -90 degrees
- moved R4 79.1 mm to (104.1, 101.6), turned to 90 degrees
- moved D3 76.4 mm to (101.6, 105.4), turned to -90 degrees
- moved R8 70.4 mm to (109.2, 101.6), turned to 90 degrees
- moved D5 70.4 mm to (109.2, 105.4), turned to -90 degrees
- moved R3 69.4 mm to (106.7, 101.6), turned to 90 degrees
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Routing:
- net /CLK: track 118.7 -> 312.7 mm, vias 0 -> 8
- net /B0: track 23.8 -> 216.3 mm, vias 2 -> 5
- net /B1: track 62.8 -> 200.8 mm, vias 11 -> 14
- net /B2: track 47.4 -> 174.8 mm, vias 2 -> 4
- net /RST: track 90.0 -> 198.7 mm, vias 0 -> 8
- net /DW: track 16.8 -> 107.1 mm, vias 6 -> 7
- net /UP: track 10.5 -> 96.5 mm, vias 4 -> 9
- net /!B1: track 29.3 -> 104.5 mm, vias 7 -> 8
- net /B3: track 45.3 -> 118.3 mm, vias 0 -> 2
- net +3V3: track 0.00 -> 66.6 mm, vias 0 -> 69
- net /!B0: track 66.2 -> 132.0 mm, vias 3 -> 4
- net /!B2: track 27.3 -> 89.6 mm, vias 5 -> 6
- net GND: track 74.3 -> 97.3 mm, vias 71 -> 86
- net /!B3: track 22.3 -> 6.85 mm, vias 3 -> 0
- net /Q_13: track 10.1 -> 19.0 mm, vias 0 -> 2
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- added copper zone on In2.Cu, net +3V3
- added copper zone on In1.Cu, net GND
Other:
- copper layers 2 -> 4
- board text added: "CLK"
- board text added: "D0"
- board text added: "D1"
- board text added: "D2"
- board text added: "D3"
- board text added: "DW"
- board text added: "PWR"
- board text added: "RST"
- board text added: "UP"
