File: Hardware/Counter/Counter.kicad_sch (KiCad schematic)
At the start: 19 parts

Commit message: started layout
Parts:
- added D5, D6: LED_Small, LED_SMD:LED_0805_2012Metric, symbol Device:LED_Small
- added R8, R9: 330R, Resistor_SMD:R_0805_2012Metric, symbol Device:R_Small_US
- J2: renamed from J?; footprint Custom_Vertical_1x_2.54mm_Pin_Header:PinHeader_1x04_P2.54mm_Vertical -> Custom_Vertical_1x_2.54mm_Pin_Header:PinHeader_1x05_P2.54mm_Vertical; symbol Connector_Generic:Conn_01x04 -> Connector_Generic:Conn_01x05
- RV1: renamed from RV?; footprint (none) -> Potentiometer_SMD:Potentiometer_Bourns_TC33X_Vertical
- gave numbers to parts that had none: 17
Connections:
- net +3V3: now also D6.2 (A)
- net B0: now also J2.2 (Pin_2); no longer J2.1 (Pin_1)
- net B1: now also J2.3 (Pin_3); no longer J2.2 (Pin_2)
- net B2: now also J2.4 (Pin_4); no longer J2.3 (Pin_3)
- net B3: now also J2.5 (Pin_5); no longer J2.4 (Pin_4)
- net CLK: now also J2.1 (Pin_1), D5.2 (A)
- net GND: now also R8.2, R9.2
- new net: D5.1 (K), R8.1
- new net: D6.1 (K), R9.1
Other:
- moved on the sheet: D1, D2, D3, D4, R1, R2, R3, R4, R5, R7, SW1, SW2

Commit message: bit 3 complete
Parts:
- added R10: 10K, Resistor_SMD:R_0805_2012Metric, symbol Device:R_Small_US
- added SW3: SW_Push, Button_Switch_SMD:SW_SPST_TL3342, symbol Switch:SW_Push
Connections:
- net GND: now also R10.1, SW3.1
- net RST: now also R10.2, SW3.2
Changed lines of the file:
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@@
   (junction (at 180.34 101.6) (diameter 1.016) (color 0 0 0 0))
   (junction (at 180.34 124.46) (diameter 1.016) (color 0 0 0 0))
+  (junction (at 180.34 144.78) (diameter 1.016) (color 0 0 0 0))
   (junction (at 216.535 131.445) (diameter 1.016) (color 0 0 0 0))
   (junction (at 216.535 158.115) (diameter 1.016) (color 0 0 0 0))
@@
     (stroke (width 0) (type solid) (color 0 0 0 0))
   )
+  (wire (pts (xy 158.75 144.78) (xy 158.75 148.59))
+    (stroke (width 0) (type solid) (color 0 0 0 0))
+  )
   (wire (pts (xy 159.385 40.64) (xy 167.64 40.64))
     (stroke (width 0) (type solid) (color 0 0 0 0))
@@
     (stroke (width 0) (type solid) (color 0 0 0 0))
   )
+  (wire (pts (xy 164.465 144.78) (xy 158.75 144.78))
+    (stroke (width 0) (type solid) (color 0 0 0 0))
+  )
   (wire (pts (xy 167.64 40.64) (xy 167.64 45.72))
     (stroke (width 0) (type solid) (color 0 0 0 0))
@@
     (stroke (width 0) (type solid) (color 0 0 0 0))
   )
+  (wire (pts (xy 174.625 144.78) (xy 180.34 144.78))
+    (stroke (width 0) (type solid) (color 0 0 0 0))
+  )
   (wire (pts (xy 180.34 89.535) (xy 180.34 92.71))
     (stroke (width 0) (type solid) (color 0 0 0 0))
@@
   )
   (wire (pts (xy 180.34 124.46) (xy 188.595 124.46))
+    (stroke (width 0) (type solid) (color 0 0 0 0))
+  )
+  (wire (pts (xy 180.34 144.78) (xy 188.595 144.78))
+    (stroke (width 0) (type solid) (color 0 0 0 0))
+  )
+  (wire (pts (xy 180.34 148.59) (xy 180.34 144.78))
+    (stroke (width 0) (type solid) (color 0 0 0 0))
+  )
+  (wire (pts (xy 180.34 156.845) (xy 180.34 153.67))
+    (stroke (width 0) (type solid) (color 0 0 0 0))
+  )
+  (wire (pts (xy 180.34 156.845) (xy 180.34 158.115))
     (stroke (width 0) (type solid) (color 0 0 0 0))
   )
@@
     (effects (font (size 1.27 1.27)) (justify right bottom))
   )
+  (label "RST" (at 188.595 144.78 180)
+    (effects (font (size 1.27 1.27)) (justify right bottom))
+  )
   (label "B0" (at 193.675 86.36 270)
     (effects (font (size 1.27 1.27)) (justify right bottom))
@@
     )
   )
+  (symbol (lib_id "power:GND") (at 158.75 148.59 0) (unit 1)
+    (in_bom yes) (on_board yes)
+    (property "Reference" "#PWR0187" (id 0) (at 158.75 154.94 0)
+      (effects (font (size 1.27 1.27)) hide)
+    )
+    (property "Value" "GND" (id 1) (at 159.385 153.67 0))
+    (property "Footprint" "" (id 2) (at 158.75 148.59 0)
+      (effects (font (size 1.27 1.27)) hide)
+    )
+    (property "Datasheet" "" (id 3) (at 158.75 148.59 0)
+      (effects (font (size 1.27 1.27)) hide)
+    )
+  )
+  (symbol (lib_id "power:GND") (at 180.34 158.115 0) (unit 1)
+    (in_bom yes) (on_board yes)
+    (property "Reference" "#PWR0201" (id 0) (at 180.34 164.465 0)
+      (effects (font (size 1.27 1.27)) hide)
+    )
+    (property "Value" "GND" (id 1) (at 180.975 163.195 0))
+    (property "Footprint" "" (id 2) (at 180.34 158.115 0)
+      (effects (font (size 1.27 1.27)) hide)
+    )
+    (property "Datasheet" "" (id 3) (at 180.34 158.115 0)
+      (effects (font (size 1.27 1.27)) hide)
+    )
+  )
   (symbol (lib_id "power:GND") (at 193.675 112.395 0) (unit 1)
     (in_bom yes) (on_board yes)
@@
     )
     (property "Datasheet" "~" (id 3) (at 180.34 118.11 0)
+      (effects (font (size 1.27 1.27)) hide)
+    )
+  )
+  (symbol (lib_id "Device:R_Small_US") (at 180.34 151.13 180) (unit 1)
+    (in_bom yes) (on_board yes)
+    (property "Reference" "R10" (id 0) (at 178.435 152.4 0)
+      (effects (font (size 1.27 1.27)) (justify left))
+    )
+    (property "Value" "10K" (id 1) (at 178.435 151.13 0)
+      (effects (font (size 1.27 1.27)) (justify left))
+    )
+    (property "Footprint" "Resistor_SMD:R_0805_2012Metric" (id 2) (at 180.34 151.13 0)
+      (effects (font (size 1.27 1.27)) hide)
+    )
+    (property "Datasheet" "~" (id 3) (at 180.34 151.13 0)
       (effects (font (size 1.27 1.27)) hide)
     )
@@
     )
     (property "Datasheet" "~" (id 3) (at 169.545 119.38 0)
+      (effects (font (size 1.27 1.27)) hide)
+    )
+  )
+  (symbol (lib_id "Switch:SW_Push") (at 169.545 144.78 0) (unit 1)
+    (in_bom yes) (on_board yes)
+    (property "Reference" "SW3" (id 0) (at 169.545 137.16 0))
+    (property "Value" "SW_Push" (id 1) (at 169.545 139.7 0))
+    (property "Footprint" "Button_Switch_SMD:SW_SPST_TL3342" (id 2) (at 169.545 139.7 0)
+      (effects (font (size 1.27 1.27)) hide)
+    )
+    (property "Datasheet" "~" (id 3) (at 169.545 139.7 0)
       (effects (font (size 1.27 1.27)) hide)
     )
@@
       (reference "#PWR0117") (unit 1) (value "GND") (footprint "")
     )
+    (path "/413165c3-66b8-4e0a-bc5e-9303cbd423ae"
+      (reference "#PWR0187") (unit 1) (value "GND") (footprint "")
+    )
+    (path "/c8c74a73-c615-4e2d-95f9-63b09304ca12"
+      (reference "#PWR0201") (unit 1) (value "GND") (footprint "")
+    )
     (path "/4ad8ee92-e07e-4007-8d7e-e0ef1f284363"
       (reference "C1") (unit 1) (value "10nF") (footprint "Capacitor_SMD:C_0805_2012Metric")
@@
       (reference "R9") (unit 1) (value "330R") (footprint "Resistor_SMD:R_0805_2012Metric")
     )
+    (path "/7ed218af-6153-4b22-af15-ff21f5fea6ec"
+      (reference "R10") (unit 1) (value "10K") (footprint "Resistor_SMD:R_0805_2012Metric")
+    )
     (path "/cc45df4d-38f5-4850-a31d-683438a58c63"
       (reference "RV1") (unit 1) (value "100K") (footprint "Potentiometer_SMD:Potentiometer_Bourns_TC33X_Vertical")
@@
       (reference "SW2") (unit 1) (value "SW_Push") (footprint "Button_Switch_SMD:SW_SPST_TL3342")
     )
+    (path "/f82b29e5-34a0-49e6-8083-18db6a79bd64"
+      (reference "SW3") (unit 1) (value "SW_Push") (footprint "Button_Switch_SMD:SW_SPST_TL3342")
+    )
     (path "/8ecf5c0b-d83e-46b6-a4a1-a5755482b684"
       (reference "U1") (unit 1) (value "LM555xM") (footprint "Package_SO:SOIC-8_3.9x4.9mm_P1.27mm")
@@
       (reference "#PWR0186") (unit 1) (value "GND") (footprint "")
     )
-    (path "/2adf4c48-4fb1-4622-9c7a-5ab5b9375e46/dc43a286-8151-4dca-9139-81451ecfada4"
-      (reference "#PWR0187") (unit 1) (value "GND") (footprint "")
-    )
     (path "/2adf4c48-4fb1-4622-9c7a-5ab5b9375e46/a8ddbf5d-54c4-48f6-a68b-378dc37eca4d"
       (reference "#PWR0188") (unit 1) (value "GND") (footprint "")
@@
       (reference "Q71") (unit 1) (value "FDN335N") (footprint "Package_TO_SOT_SMD:SOT-23")
     )
-    (path "/2adf4c48-4fb1-4622-9c7a-5ab5b9375e46/88aa5a6a-14e1-43ad-9537-1e70f0a90f63"
-      (reference "R10") (unit 1) (value "10K") (footprint "Resistor_SMD:R_0805_2012Metric")
-    )
     (path "/2adf4c48-4fb1-4622-9c7a-5ab5b9375e46/e78214fd-990b-4d12-9d9b-d4721fb5f0ff"
       (reference "U30") (unit 1) (value "FDN360P") (footprint "Package_TO_SOT_SMD:SOT-23")
@@
       (reference "#PWR0200") (unit 1) (value "GND") (footprint "")
     )
-    (path "/f173b2f8-43a9-4bbd-bc01-af58466556d3/dc43a286-8151-4dca-9139-81451ecfada4"
-      (reference "#PWR0201") (unit 1) (value "GND") (footprint "")
-    )
     (path "/f173b2f8-43a9-4bbd-bc01-af58466556d3/a8ddbf5d-54c4-48f6-a68b-378dc37eca4d"
       (reference "#PWR0202") (unit 1) (value "GND") (footprint "")
@@
       (reference "Q82") (unit 1) (value "FDN335N") (footprint "Package_TO_SOT_SMD:SOT-23")
     )
-    (path "/f173b2f8-43a9-4bbd-bc01-af58466556d3/88aa5a6a-14e1-43ad-9537-1e70f0a90f63"
-      (reference "R11") (unit 1) (value "10K") (footprint "Resistor_SMD:R_0805_2012Metric")
-    )
     (path "/f173b2f8-43a9-4bbd-bc01-af58466556d3/e78214fd-990b-4d12-9d9b-d4721fb5f0ff"
       (reference "U37") (unit 1) (value "FDN360P") (footprint "Package_TO_SOT_SMD:SOT-23")
@@
       (reference "#PWR0204") (unit 1) (value "GND") (footprint "")
     )
-    (path "/1b4c7cb5-bebb-49c1-9a9b-fd15983460e2/dc43a286-8151-4dca-9139-81451ecfada4"
-      (reference "#PWR0205") (unit 1) (value "GND") (footprint "")
-    )
     (path "/1b4c7cb5-bebb-49c1-9a9b-fd15983460e2/a8ddbf5d-54c4-48f6-a68b-378dc37eca4d"
       (reference "#PWR0206") (unit 1) (value "GND") (footprint "")
@@
       (reference "Q85") (unit 1) (value "FDN335N") (footprint "Package_TO_SOT_SMD:SOT-23")
     )
-    (path "/1b4c7cb5-bebb-49c1-9a9b-fd15983460e2/88aa5a6a-14e1-43ad-9537-1e70f0a90f63"
-      (reference "R12") (unit 1) (value "10K") (footprint "Resistor_SMD:R_0805_2012Metric")
-    )
     (path "/1b4c7cb5-bebb-49c1-9a9b-fd15983460e2/e78214fd-990b-4d12-9d9b-d4721fb5f0ff"
       (reference "U40") (unit 1) (value "FDN360P") (footprint "Package_TO_SOT_SMD:SOT-23")
@@
       (reference "#PWR0257") (unit 1) (value "GND") (footprint "")
     )
-    (path "/ae8a0611-1461-4394-8140-590c6cad4b3f/dc43a286-8151-4dca-9139-81451ecfada4"
-      (reference "#PWR0258") (unit 1) (value "GND") (footprint "")
-    )
     (path "/ae8a0611-1461-4394-8140-590c6cad4b3f/a8ddbf5d-54c4-48f6-a68b-378dc37eca4d"
       (reference "#PWR0259") (unit 1) (value "GND") (footprint "")
@@
       (reference "Q131") (unit 1) (value "FDN335N") (footprint "Package_TO_SOT_SMD:SOT-23")
     )
-    (path "/ae8a0611-1461-4394-8140-590c6cad4b3f/88aa5a6a-14e1-43ad-9537-1e70f0a90f63"
-      (reference "R13") (unit 1) (value "10K") (footprint "Resistor_SMD:R_0805_2012Metric")
-    )
     (path "/ae8a0611-1461-4394-8140-590c6cad4b3f/e78214fd-990b-4d12-9d9b-d4721fb5f0ff"

Commit message: kicad updates
Parts:
- J1: Spice_Model (none) -> dc 3.3; Spice_Netlist_Enabled (none) -> Y; Spice_Primitive (none) -> I
- SW1: Spice_Model (none) -> ac 3.3 pulse(0 3.3 1n 1n 1n 1n 2n); Spice_Netlist_Enabled (none) -> Y; Spice_Primitive (none) -> I
Changed lines of the file:
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@@
     (stroke (width 0) (type solid) (color 0 0 0 0))
   )
-  (wire (pts (xy 180.34 156.845) (xy 180.34 153.67))
-    (stroke (width 0) (type solid) (color 0 0 0 0))
-  )
-  (wire (pts (xy 180.34 156.845) (xy 180.34 158.115))
+  (wire (pts (xy 180.34 153.67) (xy 180.34 158.115))
     (stroke (width 0) (type solid) (color 0 0 0 0))
   )
@@
       (effects (font (size 1.27 1.27)) hide)
     )
+    (property "Spice_Primitive" "I" (id 4) (at 271.78 128.905 0)
+      (effects (font (size 1.27 1.27)) hide)
+    )
+    (property "Spice_Model" "dc 3.3" (id 5) (at 271.78 128.905 0)
+      (effects (font (size 1.27 1.27)) hide)
+    )
+    (property "Spice_Netlist_Enabled" "Y" (id 6) (at 271.78 128.905 0)
+      (effects (font (size 1.27 1.27)) hide)
+    )
   )
   (symbol (lib_id "Switch:SW_Push") (at 169.545 101.6 0) (unit 1)
@@
       (effects (font (size 1.27 1.27)) hide)
     )
+    (property "Spice_Primitive" "I" (id 4) (at 169.545 101.6 0)
+      (effects (font (size 1.27 1.27)) hide)
+    )
+    (property "Spice_Model" "ac 3.3 pulse(0 3.3 1n 1n 1n 1n 2n)" (id 5) (at 169.545 101.6 0)
+      (effects (font (size 1.27 1.27)) hide)
+    )
+    (property "Spice_Netlist_Enabled" "Y" (id 6) (at 169.545 101.6 0)
+      (effects (font (size 1.27 1.27)) hide)
+    )
