File: Hardware/Counter/FF.kicad_sch (KiCad schematic)
At the start: 10 parts

Commit message: started layout
Parts:
- gave numbers to parts that had none: 10
Changed lines of the file:
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@@
   (symbol (lib_id "power:+3V3") (at 57.15 76.835 0)
     (in_bom yes) (on_board yes)
-    (property "Reference" "#PWR?" (id 0) (at 57.15 80.645 0)
+    (property "Reference" "#PWR0210" (id 0) (at 57.15 80.645 0)
       (effects (font (size 1.27 1.27)) hide)
     )
@@
   (symbol (lib_id "power:+3V3") (at 153.035 76.2 0)
     (in_bom yes) (on_board yes)
-    (property "Reference" "#PWR?" (id 0) (at 153.035 80.01 0)
+    (property "Reference" "#PWR0208" (id 0) (at 153.035 80.01 0)
       (effects (font (size 1.27 1.27)) hide)
     )
@@
   (symbol (lib_id "power:+3V3") (at 177.165 76.2 0)
     (in_bom yes) (on_board yes)
-    (property "Reference" "#PWR?" (id 0) (at 177.165 80.01 0)
+    (property "Reference" "#PWR0209" (id 0) (at 177.165 80.01 0)
       (effects (font (size 1.27 1.27)) hide)
     )
@@
   (symbol (lib_id "power:GND") (at 57.15 122.555 0)
     (in_bom yes) (on_board yes)
-    (property "Reference" "#PWR?" (id 0) (at 57.15 128.905 0)
+    (property "Reference" "#PWR0211" (id 0) (at 57.15 128.905 0)
       (effects (font (size 1.27 1.27)) hide)
     )
@@
   (symbol (lib_id "power:GND") (at 153.035 121.92 0)
     (in_bom yes) (on_board yes)
-    (property "Reference" "#PWR?" (id 0) (at 153.035 128.27 0)
+    (property "Reference" "#PWR0213" (id 0) (at 153.035 128.27 0)
       (effects (font (size 1.27 1.27)) hide)
     )
@@
   (symbol (lib_id "power:GND") (at 177.165 121.92 0)
     (in_bom yes) (on_board yes)
-    (property "Reference" "#PWR?" (id 0) (at 177.165 128.27 0)
+    (property "Reference" "#PWR0212" (id 0) (at 177.165 128.27 0)
       (effects (font (size 1.27 1.27)) hide)
     )
@@
   (symbol (lib_id "Custom_Transistors:FDN360P") (at 57.15 89.535 0)
     (in_bom yes) (on_board yes)
-    (property "Reference" "U?" (id 0) (at 60.96 88.265 0)
+    (property "Reference" "U43" (id 0) (at 60.96 88.265 0)
       (effects (font (size 1.27 1.27)) (justify left))
     )
@@
   (symbol (lib_id "Custom_Transistors:FDN335N") (at 57.15 109.855 0)
     (in_bom yes) (on_board yes)
-    (property "Reference" "Q?" (id 0) (at 59.69 111.125 0)
+    (property "Reference" "Q86" (id 0) (at 59.69 111.125 0)
       (effects (font (size 1.27 1.27)) (justify left))
     )
@@
   (symbol (lib_id "Custom_Transistors:FDN360P") (at 116.205 88.9 90) (mirror x)
     (in_bom yes) (on_board yes)
-    (property "Reference" "U?" (id 0) (at 118.11 95.25 90)
+    (property "Reference" "U44" (id 0) (at 118.11 95.25 90)
       (effects (font (size 1.27 1.27)) (justify left))
     )
@@
   (symbol (lib_id "Custom_Transistors:FDN335N") (at 116.205 109.22 270) (mirror x)
     (in_bom yes) (on_board yes)
-    (property "Reference" "Q?" (id 0) (at 115.57 103.505 90)
+    (property "Reference" "Q87" (id 0) (at 115.57 103.505 90)
       (effects (font (size 1.27 1.27)) (justify left))
     )
@@
   (symbol (lib_id "Custom_Transistors:FDN360P") (at 153.035 88.9 0)
     (in_bom yes) (on_board yes)
-    (property "Reference" "U?" (id 0) (at 156.845 87.63 0)
+    (property "Reference" "U45" (id 0) (at 156.845 87.63 0)
       (effects (font (size 1.27 1.27)) (justify left))
     )
@@
   (symbol (lib_id "Custom_Transistors:FDN335N") (at 153.035 109.22 0)
     (in_bom yes) (on_board yes)
-    (property "Reference" "Q?" (id 0) (at 155.575 110.49 0)
+    (property "Reference" "Q88" (id 0) (at 155.575 110.49 0)
       (effects (font (size 1.27 1.27)) (justify left))
     )
@@
   (symbol (lib_id "Custom_Transistors:FDN360P") (at 160.02 136.525 270)
     (in_bom yes) (on_board yes)
-    (property "Reference" "U?" (id 0) (at 158.115 142.875 90)
+    (property "Reference" "U46" (id 0) (at 158.115 142.875 90)
       (effects (font (size 1.27 1.27)) (justify left))
     )
@@
   (symbol (lib_id "Custom_Transistors:FDN335N") (at 160.02 156.845 90)
     (in_bom yes) (on_board yes)
-    (property "Reference" "Q?" (id 0) (at 160.655 151.13 90)
+    (property "Reference" "Q89" (id 0) (at 160.655 151.13 90)
       (effects (font (size 1.27 1.27)) (justify left))
     )
@@
   (symbol (lib_id "Custom_Transistors:FDN360P") (at 177.165 88.9 0)
     (in_bom yes) (on_board yes)
-    (property "Reference" "U?" (id 0) (at 180.975 87.63 0)
+    (property "Reference" "U47" (id 0) (at 180.975 87.63 0)
       (effects (font (size 1.27 1.27)) (justify left))
     )
@@
   (symbol (lib_id "Custom_Transistors:FDN335N") (at 177.165 109.22 0)
     (in_bom yes) (on_board yes)
-    (property "Reference" "Q?" (id 0) (at 179.705 110.49 0)
-      (effects (font (size 1.27 1.27)) (justify left))
-    )
+    (property "Reference" "Q90" (id 0) (at 179.705 110.49 0)
+      (effects (font (size 1.27 1.27)) (justify left))
+    )

Commit message: working on connectin bits together
Parts:
- renumbered Q90 to Q100, Q86 to Q96, Q87 to Q97, Q88 to Q98, Q89 to Q99, U43 to U53, U44 to U54, U45 to U55, U46 to U56, U47 to U57
Changed lines of the file:
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@@
   (symbol (lib_id "power:+3V3") (at 57.15 76.835 0)
     (in_bom yes) (on_board yes)
-    (property "Reference" "#PWR0263" (id 0) (at 57.15 80.645 0)
+    (property "Reference" "#PWR0222" (id 0) (at 57.15 80.645 0)
       (effects (font (size 1.27 1.27)) hide)
     )
@@
   (symbol (lib_id "power:+3V3") (at 153.035 76.2 0)
     (in_bom yes) (on_board yes)
-    (property "Reference" "#PWR0261" (id 0) (at 153.035 80.01 0)
+    (property "Reference" "#PWR0220" (id 0) (at 153.035 80.01 0)
       (effects (font (size 1.27 1.27)) hide)
     )
@@
   (symbol (lib_id "power:+3V3") (at 177.165 76.2 0)
     (in_bom yes) (on_board yes)
-    (property "Reference" "#PWR0262" (id 0) (at 177.165 80.01 0)
+    (property "Reference" "#PWR0221" (id 0) (at 177.165 80.01 0)
       (effects (font (size 1.27 1.27)) hide)
     )
@@
   (symbol (lib_id "power:GND") (at 57.15 122.555 0)
     (in_bom yes) (on_board yes)
-    (property "Reference" "#PWR0264" (id 0) (at 57.15 128.905 0)
+    (property "Reference" "#PWR0223" (id 0) (at 57.15 128.905 0)
       (effects (font (size 1.27 1.27)) hide)
     )
@@
   (symbol (lib_id "power:GND") (at 153.035 121.92 0)
     (in_bom yes) (on_board yes)
-    (property "Reference" "#PWR0266" (id 0) (at 153.035 128.27 0)
+    (property "Reference" "#PWR0225" (id 0) (at 153.035 128.27 0)
       (effects (font (size 1.27 1.27)) hide)
     )
@@
   (symbol (lib_id "power:GND") (at 177.165 121.92 0)
     (in_bom yes) (on_board yes)
-    (property "Reference" "#PWR0265" (id 0) (at 177.165 128.27 0)
+    (property "Reference" "#PWR0224" (id 0) (at 177.165 128.27 0)
       (effects (font (size 1.27 1.27)) hide)
     )
@@
   (symbol (lib_name "Custom_Transistors:FDN360P_1") (lib_id "Custom_Transistors:FDN360P") (at 57.15 89.535 0)
     (in_bom yes) (on_board yes)
-    (property "Reference" "U43" (id 0) (at 60.96 88.265 0)
+    (property "Reference" "U53" (id 0) (at 60.96 88.265 0)
       (effects (font (size 1.27 1.27)) (justify left))
     )
@@
   (symbol (lib_id "Custom_Transistors:FDN335N") (at 57.15 109.855 0)
     (in_bom yes) (on_board yes)
-    (property "Reference" "Q86" (id 0) (at 59.69 111.125 0)
+    (property "Reference" "Q96" (id 0) (at 59.69 111.125 0)
       (effects (font (size 1.27 1.27)) (justify left))
     )
@@
   (symbol (lib_name "Custom_Transistors:FDN360P_2") (lib_id "Custom_Transistors:FDN360P") (at 116.205 88.9 90) (mirror x)
     (in_bom yes) (on_board yes)
-    (property "Reference" "U44" (id 0) (at 118.11 95.25 90)
+    (property "Reference" "U54" (id 0) (at 118.11 95.25 90)
       (effects (font (size 1.27 1.27)) (justify left))
     )
@@
   (symbol (lib_id "Custom_Transistors:FDN335N") (at 116.205 109.22 270) (mirror x)
     (in_bom yes) (on_board yes)
-    (property "Reference" "Q87" (id 0) (at 115.57 103.505 90)
+    (property "Reference" "Q97" (id 0) (at 115.57 103.505 90)
       (effects (font (size 1.27 1.27)) (justify left))
     )
@@
   (symbol (lib_name "Custom_Transistors:FDN360P_3") (lib_id "Custom_Transistors:FDN360P") (at 153.035 88.9 0)
     (in_bom yes) (on_board yes)
-    (property "Reference" "U45" (id 0) (at 156.845 87.63 0)
+    (property "Reference" "U55" (id 0) (at 156.845 87.63 0)
       (effects (font (size 1.27 1.27)) (justify left))
     )
@@
   (symbol (lib_id "Custom_Transistors:FDN335N") (at 153.035 109.22 0)
     (in_bom yes) (on_board yes)
-    (property "Reference" "Q88" (id 0) (at 155.575 110.49 0)
+    (property "Reference" "Q98" (id 0) (at 155.575 110.49 0)
       (effects (font (size 1.27 1.27)) (justify left))
     )
@@
   (symbol (lib_name "Custom_Transistors:FDN360P_4") (lib_id "Custom_Transistors:FDN360P") (at 160.02 136.525 270)
     (in_bom yes) (on_board yes)
-    (property "Reference" "U46" (id 0) (at 158.115 142.875 90)
+    (property "Reference" "U56" (id 0) (at 158.115 142.875 90)
       (effects (font (size 1.27 1.27)) (justify left))
     )
@@
   (symbol (lib_id "Custom_Transistors:FDN335N") (at 160.02 156.845 90)
     (in_bom yes) (on_board yes)
-    (property "Reference" "Q89" (id 0) (at 160.655 151.13 90)
+    (property "Reference" "Q99" (id 0) (at 160.655 151.13 90)
       (effects (font (size 1.27 1.27)) (justify left))
     )
@@
   (symbol (lib_id "Custom_Transistors:FDN360P") (at 177.165 88.9 0)
     (in_bom yes) (on_board yes)
-    (property "Reference" "U47" (id 0) (at 180.975 87.63 0)
+    (property "Reference" "U57" (id 0) (at 180.975 87.63 0)
       (effects (font (size 1.27 1.27)) (justify left))
     )
@@
   (symbol (lib_id "Custom_Transistors:FDN335N") (at 177.165 109.22 0)
     (in_bom yes) (on_board yes)
-    (property "Reference" "Q90" (id 0) (at 179.705 110.49 0)
-      (effects (font (size 1.27 1.27)) (justify left))
-    )
+    (property "Reference" "Q100" (id 0) (at 179.705 110.49 0)
+      (effects (font (size 1.27 1.27)) (justify left))
+    )

Commit message: kicad updates
Parts:
- renumbered Q96 to Q132, Q97 to Q133, Q98 to Q134, Q99 to Q135, Q100 to Q136, U53 to U75, U54 to U76, U55 to U77, U56 to U78, U57 to U79
Changed lines of the file:
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@@
   (symbol (lib_id "power:+3V3") (at 57.15 76.835 0)
     (in_bom yes) (on_board yes)
-    (property "Reference" "#PWR0222" (id 0) (at 57.15 80.645 0)
+    (property "Reference" "#PWR0263" (id 0) (at 57.15 80.645 0)
       (effects (font (size 1.27 1.27)) hide)
     )
@@
   (symbol (lib_id "power:+3V3") (at 153.035 76.2 0)
     (in_bom yes) (on_board yes)
-    (property "Reference" "#PWR0220" (id 0) (at 153.035 80.01 0)
+    (property "Reference" "#PWR0261" (id 0) (at 153.035 80.01 0)
       (effects (font (size 1.27 1.27)) hide)
     )
@@
   (symbol (lib_id "power:+3V3") (at 177.165 76.2 0)
     (in_bom yes) (on_board yes)
-    (property "Reference" "#PWR0221" (id 0) (at 177.165 80.01 0)
+    (property "Reference" "#PWR0262" (id 0) (at 177.165 80.01 0)
       (effects (font (size 1.27 1.27)) hide)
     )
@@
   (symbol (lib_id "power:GND") (at 57.15 122.555 0)
     (in_bom yes) (on_board yes)
-    (property "Reference" "#PWR0223" (id 0) (at 57.15 128.905 0)
+    (property "Reference" "#PWR0264" (id 0) (at 57.15 128.905 0)
       (effects (font (size 1.27 1.27)) hide)
     )
@@
   (symbol (lib_id "power:GND") (at 153.035 121.92 0)
     (in_bom yes) (on_board yes)
-    (property "Reference" "#PWR0225" (id 0) (at 153.035 128.27 0)
+    (property "Reference" "#PWR0266" (id 0) (at 153.035 128.27 0)
       (effects (font (size 1.27 1.27)) hide)
     )
@@
   (symbol (lib_id "power:GND") (at 177.165 121.92 0)
     (in_bom yes) (on_board yes)
-    (property "Reference" "#PWR0224" (id 0) (at 177.165 128.27 0)
+    (property "Reference" "#PWR0265" (id 0) (at 177.165 128.27 0)
       (effects (font (size 1.27 1.27)) hide)
     )
@@
   (symbol (lib_name "Custom_Transistors:FDN360P_1") (lib_id "Custom_Transistors:FDN360P") (at 57.15 89.535 0)
     (in_bom yes) (on_board yes)
-    (property "Reference" "U53" (id 0) (at 60.96 88.265 0)
+    (property "Reference" "U75" (id 0) (at 60.96 88.265 0)
       (effects (font (size 1.27 1.27)) (justify left))
     )
@@
   (symbol (lib_id "Custom_Transistors:FDN335N") (at 57.15 109.855 0)
     (in_bom yes) (on_board yes)
-    (property "Reference" "Q96" (id 0) (at 59.69 111.125 0)
+    (property "Reference" "Q132" (id 0) (at 59.69 111.125 0)
       (effects (font (size 1.27 1.27)) (justify left))
     )
@@
   (symbol (lib_name "Custom_Transistors:FDN360P_2") (lib_id "Custom_Transistors:FDN360P") (at 116.205 88.9 90) (mirror x)
     (in_bom yes) (on_board yes)
-    (property "Reference" "U54" (id 0) (at 118.11 95.25 90)
+    (property "Reference" "U76" (id 0) (at 118.11 95.25 90)
       (effects (font (size 1.27 1.27)) (justify left))
     )
@@
   (symbol (lib_id "Custom_Transistors:FDN335N") (at 116.205 109.22 270) (mirror x)
     (in_bom yes) (on_board yes)
-    (property "Reference" "Q97" (id 0) (at 115.57 103.505 90)
+    (property "Reference" "Q133" (id 0) (at 115.57 103.505 90)
       (effects (font (size 1.27 1.27)) (justify left))
     )
@@
   (symbol (lib_name "Custom_Transistors:FDN360P_3") (lib_id "Custom_Transistors:FDN360P") (at 153.035 88.9 0)
     (in_bom yes) (on_board yes)
-    (property "Reference" "U55" (id 0) (at 156.845 87.63 0)
+    (property "Reference" "U77" (id 0) (at 156.845 87.63 0)
       (effects (font (size 1.27 1.27)) (justify left))
     )
@@
   (symbol (lib_id "Custom_Transistors:FDN335N") (at 153.035 109.22 0)
     (in_bom yes) (on_board yes)
-    (property "Reference" "Q98" (id 0) (at 155.575 110.49 0)
+    (property "Reference" "Q134" (id 0) (at 155.575 110.49 0)
       (effects (font (size 1.27 1.27)) (justify left))
     )
@@
   (symbol (lib_name "Custom_Transistors:FDN360P_4") (lib_id "Custom_Transistors:FDN360P") (at 160.02 136.525 270)
     (in_bom yes) (on_board yes)
-    (property "Reference" "U56" (id 0) (at 158.115 142.875 90)
+    (property "Reference" "U78" (id 0) (at 158.115 142.875 90)
       (effects (font (size 1.27 1.27)) (justify left))
     )
@@
   (symbol (lib_id "Custom_Transistors:FDN335N") (at 160.02 156.845 90)
     (in_bom yes) (on_board yes)
-    (property "Reference" "Q99" (id 0) (at 160.655 151.13 90)
+    (property "Reference" "Q135" (id 0) (at 160.655 151.13 90)
       (effects (font (size 1.27 1.27)) (justify left))
     )
@@
   (symbol (lib_id "Custom_Transistors:FDN360P") (at 177.165 88.9 0)
     (in_bom yes) (on_board yes)
-    (property "Reference" "U57" (id 0) (at 180.975 87.63 0)
+    (property "Reference" "U79" (id 0) (at 180.975 87.63 0)
       (effects (font (size 1.27 1.27)) (justify left))
     )
@@
   (symbol (lib_id "Custom_Transistors:FDN335N") (at 177.165 109.22 0)
     (in_bom yes) (on_board yes)
-    (property "Reference" "Q100" (id 0) (at 179.705 110.49 0)
-      (effects (font (size 1.27 1.27)) (justify left))
-    )
+    (property "Reference" "Q136" (id 0) (at 179.705 110.49 0)
+      (effects (font (size 1.27 1.27)) (justify left))
+    )
